File: WiFiDuck.kicad_sch (KiCad schematic)
At the start: 11 parts, among them J1 USB_A, J2 DEBUG, U1 ESP-12F, U2 CH9328, U3 AMS1117-3.3

Commit message: v0.2.0
Fix CH9328 footprint
Parts:
- U2: footprint Package_DIP:DIP-16_W7.62mm_SMDSocket_SmallPads -> Package_SO:SOP-16_3.9x9.9mm_P1.27mm
Changed lines of the file:
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@@
       (effects (font (size 1.27 1.27)))
     )
-    (property "Footprint" "Package_DIP:DIP-16_W7.62mm_SMDSocket_SmallPads" (at 157.48 110.49 0)
+    (property "Footprint" "Package_SO:SOP-16_3.9x9.9mm_P1.27mm" (at 157.48 110.49 0)
       (effects (font (size 1.27 1.27)) hide)
     )
